File: hardware/floracarepcb.kicad_pcb (KiCad board)
At the start: 2 copper layers, 100 x 100 mm, 17 parts, among them J1 USB_C_Receptacle_USB2.0_14P, J2 Conn_01x04_Socket, J3 Conn_01x08_Socket, J4 Conn_01x04_Socket, J6 Conn_01x05_Socket, U1 AMS1117-3.3, U2 ESP32-S3-WROOM-1

Commit message: Remaking hardware directory
Parts:
- removed J3: Conn_01x08_Socket, Connector_PinHeader_2.54mm:PinHeader_1x08_P2.54mm_Vertical
- added J5: Conn_01x14_Socket, Connector_PinHeader_2.54mm:PinHeader_1x14_P2.54mm_Vertical, F.Cu at (143.4, 36.8)
- moved J4 39.6 mm to (206.4, 86.2)
- moved J2 39.1 mm to (170.4, 104.2)
- moved J6 4.00 mm to (166.4, 87.2)
- moved C6 1.63 mm to (202.4, 86.8), turned to 180 degrees
Connections:
- U2 pad 17: unconnected-(U2-IO9-Pad17) -> RES
- U2 pad 21: RES -> LED
- U2 pad 38: unconnected-(U2-IO2-Pad38) -> LIGH_SCL
- U2 pad 39: unconnected-(U2-IO1-Pad39) -> LIGHT_SDA
- U2 pad 8: unconnected-(U2-IO15-Pad8) -> DHT11
- U2 pad 9: DHT11 -> unconnected-(U2-IO16-Pad9)
Routing:
- net RES: track 0.00 -> 69.1 mm
- net SCLK: track 0.00 -> 69.0 mm, vias 0 -> 2
- net LED: track 0.00 -> 68.8 mm, vias 0 -> 2
- net MOSI: track 0.00 -> 68.7 mm, vias 0 -> 2
- net CS: track 0.00 -> 66.8 mm
- net DC: track 0.00 -> 65.2 mm, vias 0 -> 2
- net AO_SOIL: track 0.00 -> 48.5 mm, vias 0 -> 1
- net LIGH_SCL: track 0.00 -> 29.8 mm
- net LIGHT_SDA: track 0.00 -> 29.6 mm
- net DHT11: track 0.00 -> 21.1 mm, vias 0 -> 1
- net GND: track 3.53 -> 0.11 mm
- removed copper zone on B.Cu, net GND
